Commit message: 第二次

File: star_/urdf/star_.urdf (robot description, URDF)
Before this commit: robot star_, 5 links, 4 joints
Joints:
- joint j1: limit lower=0 upper=0 effort=0 velocity=0 -> lower=-3.14159 upper=3.14159 effort=10 velocity=3.14
- joint j2: limit lower=0 upper=0 effort=0 velocity=0 -> lower=-1.5708 upper=1.5708 effort=10 velocity=3.14
- joint j3: limit lower=0 upper=0 effort=0 velocity=0 -> lower=-1.5708 upper=1.5708 effort=10 velocity=3.14
- joint j4: limit lower=0 upper=0 effort=0 velocity=0 -> lower=-1.5708 upper=1.5708 effort=10 velocity=3.14
